File: KiCAD/antennaBoard/antennaBoard.kicad_pcb (KiCad board)
At the start: 4 copper layers, 59.4 x 53.8 mm, 3 parts, among them J1 Conn_Coaxial, J3 Conn_Coaxial

Commit message: Update KiCAD
Routing:
- added copper zone on B.Cu, net GND
Changed lines of the file:
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@@
 		(capping no)
 		(filling no)
+		(zone_defaults)
 		(grid_origin 157.734 101.092)
 		(pcbplotparams
@@
 		(net "GND")
 	)
+	(zone
+		(net "GND")
+		(layer "B.Cu")
+		(hatch edge 0.5)
+		(connect_pads
+			(clearance 0.5)
+		)
+		(min_thickness 0.25)
+		(fill yes
+			(thermal_gap 0.5)
+			(thermal_bridge_width 0.5)
+			(island_removal_mode 0)
+		)
+		(polygon
+			(pts
+				(xy 186.374 71.12) (xy 129.204 71.12) (xy 129.204 122.852) (xy 186.374 122.852)
+			)
+		)
+	)
 	(embedded_fonts no)
